File: pcb/output.sch (KiCad schematic (older format))
At the start: 4 parts, among them J6 CONN_01X16, U11 MCP23017

Commit message: Updating PCB
Parts:
- removed C?: 0.1uF, symbol C
- removed C?: 22uF, symbol CP
- removed J6: CONN_01X16, symbol CONN_01X16
- removed U11: MCP23017, symbol MCP23017
- added C5: 0.1uF, Capacitor_THT:C_Disc_D5.0mm_W2.5mm_P2.50mm, symbol Device:C
- added J11, J12: Conn_01x08_Male, TerminalBlock_TE-Connectivity:TerminalBlock_TE_282834-8_1x08_P2.54mm_Horizontal, symbol Connector:Conn_01x08_Male
- added U12: MCP23017-E_SP, Package_DIP:DIP-28_W7.62mm, symbol dk_Interface-I-O-Expanders:MCP23017-E_SP
Connections:
- net labels added: Out0, Out1, Out10, Out11, Out12, Out13, Out14, Out15, Out2, Out3, Out4, Out5, Out6, Out7, Out8, Out9, Pin0, Pin1, Pin10, Pin11, Pin12, Pin13, Pin14, Pin15, Pin2, Pin3, Pin4, Pin5, Pin6, Pin7, Pin8, Pin9, ~RESET
- net labels removed: OUT0, OUT1, OUT10, OUT11, OUT12, OUT13, OUT14, OUT15, OUT2, OUT3, OUT4, OUT5, OUT6, OUT7, OUT8, OUT9, OUT[0..15], RESET
- wire segments 38 -> 78
