File: pcb/opto.sch (KiCad schematic (older format))
At the start: 9 parts, among them U3 LTV-847

Commit message: latest
Parts:
- R1, R2, R3, R4: value 680 1W -> 1k 1W
Changed lines of the file:
@@
 $Descr A4 11693 8268
 encoding utf-8
-Sheet 4 45
+Sheet 3 45
 Title ""
 Date ""
@@
 AR Path="/5C211542/5C23EEB9/5C212CE3" Ref="U6"  Part="1"
 AR Path="/5C211551/5C23EEB9/5C212CE3" Ref="U11"  Part="1"
-F 0 "U11" V 5453 2672 60  0000 R CNN
+F 0 "U3" V 5453 2672 60  0000 R CNN
 F 1 "LTV-847" V 5347 2672 60  0000 R CNN
 F 2 "Package_DIP:DIP-16_W7.62mm" H 5600 3400 60  0001 L CNN
@@
 AR Path="/5C211551/5C23E138/5C2C927B" Ref="R25"  Part="1"
 AR Path="/5C211551/5C23EEB9/5C2C927B" Ref="R29"  Part="1"
-F 0 "R29" V 2443 4800 50  0000 C CNN
-F 1 "680 1W" V 2534 4800 50  0000 C CNN
+F 0 "R1" V 2443 4800 50  0000 C CNN
+F 1 "1k 1W" V 2534 4800 50  0000 C CNN
 F 2 "Resistor_THT:R_Axial_DIN0414_L11.9mm_D4.5mm_P5.08mm_Vertical" V 2580 4800 50  0001 C CNN
 F 3 "~" H 2650 4800 50  0001 C CNN
@@
 AR Path="/5C211551/5C23E138/5C2C92BD" Ref="R26"  Part="1"
 AR Path="/5C211551/5C23EEB9/5C2C92BD" Ref="R30"  Part="1"
-F 0 "R30" V 2443 5100 50  0000 C CNN
-F 1 "680 1W" V 2534 5100 50  0000 C CNN
+F 0 "R2" V 2443 5100 50  0000 C CNN
+F 1 "1k 1W" V 2534 5100 50  0000 C CNN
 F 2 "Resistor_THT:R_Axial_DIN0414_L11.9mm_D4.5mm_P5.08mm_Vertical" V 2580 5100 50  0001 C CNN
 F 3 "~" H 2650 5100 50  0001 C CNN
@@
 AR Path="/5C211551/5C23E138/5C2C92D9" Ref="R27"  Part="1"
 AR Path="/5C211551/5C23EEB9/5C2C92D9" Ref="R31"  Part="1"
-F 0 "R31" V 2443 5400 50  0000 C CNN
-F 1 "680 1W" V 2534 5400 50  0000 C CNN
+F 0 "R3" V 2443 5400 50  0000 C CNN
+F 1 "1k 1W" V 2534 5400 50  0000 C CNN
 F 2 "Resistor_THT:R_Axial_DIN0414_L11.9mm_D4.5mm_P5.08mm_Vertical" V 2580 5400 50  0001 C CNN
 F 3 "~" H 2650 5400 50  0001 C CNN
@@
 AR Path="/5C211551/5C23E138/5C2C92F3" Ref="R28"  Part="1"
 AR Path="/5C211551/5C23EEB9/5C2C92F3" Ref="R32"  Part="1"
-F 0 "R32" V 2443 5700 50  0000 C CNN
-F 1 "680 1W" V 2534 5700 50  0000 C CNN
+F 0 "R4" V 2443 5700 50  0000 C CNN
+F 1 "1k 1W" V 2534 5700 50  0000 C CNN
 F 2 "Resistor_THT:R_Axial_DIN0414_L11.9mm_D4.5mm_P5.08mm_Vertical" V 2580 5700 50  0001 C CNN
 F 3 "~" H 2650 5700 50  0001 C CNN
@@
 AR Path="/5C211551/5C23E138/5C2CC03E" Ref="#PWR043"  Part="1"
 AR Path="/5C211551/5C23EEB9/5C2CC03E" Ref="#PWR045"  Part="1"
-F 0 "#PWR045" H 6150 2750 50  0001 C CNN
+F 0 "#PWR028" H 6150 2750 50  0001 C CNN
 F 1 "GND" H 6155 2827 50  0000 C CNN
 F 2 "" H 6150 3000 50  0001 C CNN
@@
 AR Path="/5C211551/5C23E138/5C24546C" Ref="#PWR042"  Part="1"
 AR Path="/5C211551/5C23EEB9/5C24546C" Ref="#PWR044"  Part="1"
-F 0 "#PWR044" H 3000 3200 50  0001 C CNN
+F 0 "#PWR027" H 3000 3200 50  0001 C CNN
 F 1 "+12V" H 3015 3523 50  0000 C CNN
 F 2 "" H 3000 3350 50  0001 C CNN
@@
 AR Path="/5C211551/5C23E138/5C26E058" Ref="D25"  Part="1"
 AR Path="/5C211551/5C23EEB9/5C26E058" Ref="D29"  Part="1"
-F 0 "D29" V 3204 4229 50  0000 L CNN
+F 0 "D1" V 3204 4229 50  0000 L CNN
 F 1 "1N4001" V 3295 4229 50  0000 L CNN
 F 2 "Diode_THT:D_DO-41_SOD81_P10.16mm_Horizontal" H 3250 3975 50  0001 C CNN
@@
 AR Path="/5C211551/5C23E138/5C26E098" Ref="D26"  Part="1"
 AR Path="/5C211551/5C23EEB9/5C26E098" Ref="D30"  Part="1"
-F 0 "D30" V 3654 4229 50  0000 L CNN
+F 0 "D2" V 3654 4229 50  0000 L CNN
 F 1 "1N4001" V 3745 4229 50  0000 L CNN
 F 2 "Diode_THT:D_DO-41_SOD81_P10.16mm_Horizontal" H 3700 3975 50  0001 C CNN
@@
 AR Path="/5C211551/5C23E138/5C274049" Ref="D27"  Part="1"
 AR Path="/5C211551/5C23EEB9/5C274049" Ref="D31"  Part="1"
-F 0 "D31" V 4104 4229 50  0000 L CNN
+F 0 "D3" V 4104 4229 50  0000 L CNN
 F 1 "1N4001" V 4195 4229 50  0000 L CNN
 F 2 "Diode_THT:D_DO-41_SOD81_P10.16mm_Horizontal" H 4150 3975 50  0001 C CNN
@@
 AR Path="/5C211551/5C23E138/5C274050" Ref="D28"  Part="1"
 AR Path="/5C211551/5C23EEB9/5C274050" Ref="D32"  Part="1"
-F 0 "D32" V 4554 4229 50  0000 L CNN
+F 0 "D4" V 4554 4229 50  0000 L CNN
 F 1 "1N4001" V 4645 4229 50  0000 L CNN
 F 2 "Diode_THT:D_DO-41_SOD81_P10.16mm_Horizontal" H 4600 3975 50  0001 C CNN

Commit message: 4 layer PCB
Changed lines of the file:
@@
 AR Path="/5C211542/5C23EEB9/5C212CE3" Ref="U6"  Part="1"
 AR Path="/5C211551/5C23EEB9/5C212CE3" Ref="U11"  Part="1"
-F 0 "U3" V 5453 2672 60  0000 R CNN
+F 0 "U11" V 5453 2672 60  0000 R CNN
 F 1 "LTV-847" V 5347 2672 60  0000 R CNN
 F 2 "Package_DIP:DIP-16_W7.62mm" H 5600 3400 60  0001 L CNN
@@
 AR Path="/5C211551/5C23E138/5C2C927B" Ref="R25"  Part="1"
 AR Path="/5C211551/5C23EEB9/5C2C927B" Ref="R29"  Part="1"
-F 0 "R1" V 2443 4800 50  0000 C CNN
+F 0 "R29" V 2443 4800 50  0000 C CNN
 F 1 "1k 1W" V 2534 4800 50  0000 C CNN
 F 2 "Resistor_THT:R_Axial_DIN0414_L11.9mm_D4.5mm_P5.08mm_Vertical" V 2580 4800 50  0001 C CNN
@@
 AR Path="/5C211551/5C23E138/5C2C92BD" Ref="R26"  Part="1"
 AR Path="/5C211551/5C23EEB9/5C2C92BD" Ref="R30"  Part="1"
-F 0 "R2" V 2443 5100 50  0000 C CNN
+F 0 "R30" V 2443 5100 50  0000 C CNN
 F 1 "1k 1W" V 2534 5100 50  0000 C CNN
 F 2 "Resistor_THT:R_Axial_DIN0414_L11.9mm_D4.5mm_P5.08mm_Vertical" V 2580 5100 50  0001 C CNN
@@
 AR Path="/5C211551/5C23E138/5C2C92D9" Ref="R27"  Part="1"
 AR Path="/5C211551/5C23EEB9/5C2C92D9" Ref="R31"  Part="1"
-F 0 "R3" V 2443 5400 50  0000 C CNN
+F 0 "R31" V 2443 5400 50  0000 C CNN
 F 1 "1k 1W" V 2534 5400 50  0000 C CNN
 F 2 "Resistor_THT:R_Axial_DIN0414_L11.9mm_D4.5mm_P5.08mm_Vertical" V 2580 5400 50  0001 C CNN
@@
 AR Path="/5C211551/5C23E138/5C2C92F3" Ref="R28"  Part="1"
 AR Path="/5C211551/5C23EEB9/5C2C92F3" Ref="R32"  Part="1"
-F 0 "R4" V 2443 5700 50  0000 C CNN
+F 0 "R32" V 2443 5700 50  0000 C CNN
 F 1 "1k 1W" V 2534 5700 50  0000 C CNN
 F 2 "Resistor_THT:R_Axial_DIN0414_L11.9mm_D4.5mm_P5.08mm_Vertical" V 2580 5700 50  0001 C CNN
@@
 AR Path="/5C211551/5C23E138/5C2CC03E" Ref="#PWR043"  Part="1"
 AR Path="/5C211551/5C23EEB9/5C2CC03E" Ref="#PWR045"  Part="1"
-F 0 "#PWR028" H 6150 2750 50  0001 C CNN
+F 0 "#PWR045" H 6150 2750 50  0001 C CNN
 F 1 "GND" H 6155 2827 50  0000 C CNN
 F 2 "" H 6150 3000 50  0001 C CNN
@@
 AR Path="/5C211551/5C23E138/5C24546C" Ref="#PWR042"  Part="1"
 AR Path="/5C211551/5C23EEB9/5C24546C" Ref="#PWR044"  Part="1"
-F 0 "#PWR027" H 3000 3200 50  0001 C CNN
+F 0 "#PWR044" H 3000 3200 50  0001 C CNN
 F 1 "+12V" H 3015 3523 50  0000 C CNN
 F 2 "" H 3000 3350 50  0001 C CNN
@@
 AR Path="/5C211551/5C23E138/5C26E058" Ref="D25"  Part="1"
 AR Path="/5C211551/5C23EEB9/5C26E058" Ref="D29"  Part="1"
-F 0 "D1" V 3204 4229 50  0000 L CNN
+F 0 "D29" V 3204 4229 50  0000 L CNN
 F 1 "1N4001" V 3295 4229 50  0000 L CNN
 F 2 "Diode_THT:D_DO-41_SOD81_P10.16mm_Horizontal" H 3250 3975 50  0001 C CNN
@@
 AR Path="/5C211551/5C23E138/5C26E098" Ref="D26"  Part="1"
 AR Path="/5C211551/5C23EEB9/5C26E098" Ref="D30"  Part="1"
-F 0 "D2" V 3654 4229 50  0000 L CNN
+F 0 "D30" V 3654 4229 50  0000 L CNN
 F 1 "1N4001" V 3745 4229 50  0000 L CNN
 F 2 "Diode_THT:D_DO-41_SOD81_P10.16mm_Horizontal" H 3700 3975 50  0001 C CNN
@@
 AR Path="/5C211551/5C23E138/5C274049" Ref="D27"  Part="1"
 AR Path="/5C211551/5C23EEB9/5C274049" Ref="D31"  Part="1"
-F 0 "D3" V 4104 4229 50  0000 L CNN
+F 0 "D31" V 4104 4229 50  0000 L CNN
 F 1 "1N4001" V 4195 4229 50  0000 L CNN
 F 2 "Diode_THT:D_DO-41_SOD81_P10.16mm_Horizontal" H 4150 3975 50  0001 C CNN
@@
 AR Path="/5C211551/5C23E138/5C274050" Ref="D28"  Part="1"
 AR Path="/5C211551/5C23EEB9/5C274050" Ref="D32"  Part="1"
-F 0 "D4" V 4554 4229 50  0000 L CNN
+F 0 "D32" V 4554 4229 50  0000 L CNN
 F 1 "1N4001" V 4645 4229 50  0000 L CNN
 F 2 "Diode_THT:D_DO-41_SOD81_P10.16mm_Horizontal" H 4600 3975 50  0001 C CNN

Commit message: Changed some footprints, spacing out components
Parts:
- R1, R2, R3, R4: footprint Resistor_THT:R_Axial_DIN0414_L11.9mm_D4.5mm_P5.08mm_Vertical -> Resistor_THT:R_Axial_DIN0414_L11.9mm_D4.5mm_P7.62mm_Vertical
Connections:
- net In0: now also R1.1; no longer R1.2
- net In1: now also R2.1; no longer R2.2
- net In2: now also R3.1; no longer R3.2
- net In3: now also R4.1; no longer R4.2
- net at D1.2 (A), U3.2: now also R1.2; no longer R1.1
- net at D2.2 (A), U3.4: now also R2.2; no longer R2.1
- net at D3.2 (A), U3.6: now also R3.2; no longer R3.1
- net at D4.2 (A), U3.8: now also R4.2; no longer R4.1
Changed lines of the file:
@@
 AR Path="/5C211542/5C23EEB9/5C212CE3" Ref="U6"  Part="1"
 AR Path="/5C211551/5C23EEB9/5C212CE3" Ref="U11"  Part="1"
-F 0 "U11" V 5453 2672 60  0000 R CNN
+F 0 "U3" V 5453 2672 60  0000 R CNN
 F 1 "LTV-847" V 5347 2672 60  0000 R CNN
 F 2 "Package_DIP:DIP-16_W7.62mm" H 5600 3400 60  0001 L CNN
@@
 AR Path="/5C211551/5C23E138/5C2C927B" Ref="R25"  Part="1"
 AR Path="/5C211551/5C23EEB9/5C2C927B" Ref="R29"  Part="1"
-F 0 "R29" V 2443 4800 50  0000 C CNN
+F 0 "R1" V 2443 4800 50  0000 C CNN
 F 1 "1k 1W" V 2534 4800 50  0000 C CNN
-F 2 "Resistor_THT:R_Axial_DIN0414_L11.9mm_D4.5mm_P5.08mm_Vertical" V 2580 4800 50  0001 C CNN
+F 2 "Resistor_THT:R_Axial_DIN0414_L11.9mm_D4.5mm_P7.62mm_Vertical" V 2580 4800 50  0001 C CNN
 F 3 "~" H 2650 4800 50  0001 C CNN
 	1    2650 4800
-	0    1    1    0
+	0    -1   -1   0
 $EndComp
 $Comp
@@
 AR Path="/5C211551/5C23E138/5C2C92BD" Ref="R26"  Part="1"
 AR Path="/5C211551/5C23EEB9/5C2C92BD" Ref="R30"  Part="1"
-F 0 "R30" V 2443 5100 50  0000 C CNN
+F 0 "R2" V 2443 5100 50  0000 C CNN
 F 1 "1k 1W" V 2534 5100 50  0000 C CNN
-F 2 "Resistor_THT:R_Axial_DIN0414_L11.9mm_D4.5mm_P5.08mm_Vertical" V 2580 5100 50  0001 C CNN
+F 2 "Resistor_THT:R_Axial_DIN0414_L11.9mm_D4.5mm_P7.62mm_Vertical" V 2580 5100 50  0001 C CNN
 F 3 "~" H 2650 5100 50  0001 C CNN
 	1    2650 5100
-	0    1    1    0
+	0    -1   -1   0
 $EndComp
 $Comp
@@
 AR Path="/5C211551/5C23E138/5C2C92D9" Ref="R27"  Part="1"
 AR Path="/5C211551/5C23EEB9/5C2C92D9" Ref="R31"  Part="1"
-F 0 "R31" V 2443 5400 50  0000 C CNN
+F 0 "R3" V 2443 5400 50  0000 C CNN
 F 1 "1k 1W" V 2534 5400 50  0000 C CNN
-F 2 "Resistor_THT:R_Axial_DIN0414_L11.9mm_D4.5mm_P5.08mm_Vertical" V 2580 5400 50  0001 C CNN
+F 2 "Resistor_THT:R_Axial_DIN0414_L11.9mm_D4.5mm_P7.62mm_Vertical" V 2580 5400 50  0001 C CNN
 F 3 "~" H 2650 5400 50  0001 C CNN
 	1    2650 5400
-	0    1    1    0
+	0    -1   -1   0
 $EndComp
 $Comp
@@
 AR Path="/5C211551/5C23E138/5C2C92F3" Ref="R28"  Part="1"
 AR Path="/5C211551/5C23EEB9/5C2C92F3" Ref="R32"  Part="1"
-F 0 "R32" V 2443 5700 50  0000 C CNN
+F 0 "R4" V 2443 5700 50  0000 C CNN
 F 1 "1k 1W" V 2534 5700 50  0000 C CNN
-F 2 "Resistor_THT:R_Axial_DIN0414_L11.9mm_D4.5mm_P5.08mm_Vertical" V 2580 5700 50  0001 C CNN
+F 2 "Resistor_THT:R_Axial_DIN0414_L11.9mm_D4.5mm_P7.62mm_Vertical" V 2580 5700 50  0001 C CNN
 F 3 "~" H 2650 5700 50  0001 C CNN
 	1    2650 5700
-	0    1    1    0
+	0    -1   -1   0
 $EndComp
 Wire Wire Line
@@
 AR Path="/5C211551/5C23E138/5C26E058" Ref="D25"  Part="1"
 AR Path="/5C211551/5C23EEB9/5C26E058" Ref="D29"  Part="1"
-F 0 "D29" V 3204 4229 50  0000 L CNN
+F 0 "D1" V 3204 4229 50  0000 L CNN
 F 1 "1N4001" V 3295 4229 50  0000 L CNN
 F 2 "Diode_THT:D_DO-41_SOD81_P10.16mm_Horizontal" H 3250 3975 50  0001 C CNN
@@
 AR Path="/5C211551/5C23E138/5C26E098" Ref="D26"  Part="1"
 AR Path="/5C211551/5C23EEB9/5C26E098" Ref="D30"  Part="1"
-F 0 "D30" V 3654 4229 50  0000 L CNN
+F 0 "D2" V 3654 4229 50  0000 L CNN
 F 1 "1N4001" V 3745 4229 50  0000 L CNN
 F 2 "Diode_THT:D_DO-41_SOD81_P10.16mm_Horizontal" H 3700 3975 50  0001 C CNN
@@
 AR Path="/5C211551/5C23E138/5C274049" Ref="D27"  Part="1"
 AR Path="/5C211551/5C23EEB9/5C274049" Ref="D31"  Part="1"
-F 0 "D31" V 4104 4229 50  0000 L CNN
+F 0 "D3" V 4104 4229 50  0000 L CNN
 F 1 "1N4001" V 4195 4229 50  0000 L CNN
 F 2 "Diode_THT:D_DO-41_SOD81_P10.16mm_Horizontal" H 4150 3975 50  0001 C CNN
@@
 AR Path="/5C211551/5C23E138/5C274050" Ref="D28"  Part="1"
 AR Path="/5C211551/5C23EEB9/5C274050" Ref="D32"  Part="1"
-F 0 "D32" V 4554 4229 50  0000 L CNN
+F 0 "D4" V 4554 4229 50  0000 L CNN
 F 1 "1N4001" V 4645 4229 50  0000 L CNN
 F 2 "Diode_THT:D_DO-41_SOD81_P10.16mm_Horizontal" H 4600 3975 50  0001 C CNN
