File: pcb/pcb.sch (KiCad schematic (older format))
At the start: 21 parts, among them J1 Barrel_Jack, J15 Conn_01x02_Male, J2 Barrel_Jack, J3 Screw_Terminal_01x02, J4 Screw_Terminal_01x02, J5 Conn_02x05_Odd_Even, J6 Conn_01x06_Male, SW1 SW_SPDT, SW2 SW_SPDT, U1 CPC5001G

Commit message: version that went into production
Parts:
- J15: value Conn_01x02_Male -> Conn_01x04_Male; footprint Connector_PinHeader_2.54mm:PinHeader_1x02_P2.54mm_Vertical -> Connector_PinHeader_2.54mm:PinHeader_1x04_P2.54mm_Vertical; symbol Connector:Conn_01x02_Male -> Connector:Conn_01x04_Male
Connections:
- net +5V: now also J15.1 (Pin_1), SW1.1 (A)
- net GND: now also J15.4 (Pin_4), SW1.3 (C)
- net SCL: now also J15.3 (Pin_3); no longer J15.2 (Pin_2)
- net SDA: now also J15.2 (Pin_2); no longer J15.1 (Pin_1)
Other:
- moved on the sheet: SW1
Changed lines of the file:
@@
 	1    0    0    -1
 $EndComp
-Text Label 4650 3100 0    50   ~ 0
+Text Label 4550 2900 0    50   ~ 0
 PRG_MODE
 Wire Wire Line
@@
 PRG_MODE
 Wire Wire Line
-	4650 3100 5100 3100
+	4550 2900 5000 2900
 $Comp
 L Switch:SW_SPDT SW1
 U 1 1 5C2A8AB1
-P 5300 3100
-F 0 "SW1" H 5300 3385 50  0000 C CNN
-F 1 "SW_SPDT" H 5300 3294 50  0000 C CNN
-F 2 "digikey-footprints:Switch_Slide_11.6x4mm_EG1218" H 5300 3100 50  0001 C CNN
-F 3 "" H 5300 3100 50  0001 C CNN
-	1    5300 3100
+P 5200 2900
+F 0 "SW1" H 5200 3185 50  0000 C CNN
+F 1 "SW_SPDT" H 5200 3094 50  0000 C CNN
+F 2 "digikey-footprints:Switch_Slide_11.6x4mm_EG1218" H 5200 2900 50  0001 C CNN
+F 3 "" H 5200 2900 50  0001 C CNN
+	1    5200 2900
 	1    0    0    -1
 $EndComp
@@
 $EndComp
 $Comp
-L Connector:Conn_01x02_Male J15
+L Connector:Conn_01x04_Male J15
 U 1 1 5C4DCA45
-P 5200 4200
-F 0 "J15" H 5306 4378 50  0000 C CNN
-F 1 "Conn_01x02_Male" H 5306 4287 50  0000 C CNN
-F 2 "Connector_PinHeader_2.54mm:PinHeader_1x02_P2.54mm_Vertical" H 5200 4200 50  0001 C CNN
-F 3 "~" H 5200 4200 50  0001 C CNN
-	1    5200 4200
-	1    0    0    -1
-$EndComp
-Wire Wire Line
-	5400 4200 5500 4200
-Wire Wire Line
-	5400 4300 5500 4300
-Text GLabel 5500 4200 2    50   Input ~ 0
+P 5150 3950
+F 0 "J15" H 5256 4128 50  0000 C CNN
+F 1 "Conn_01x04_Male" H 5300 3650 50  0000 C CNN
+F 2 "Connector_PinHeader_2.54mm:PinHeader_1x04_P2.54mm_Vertical" H 5150 3950 50  0001 C CNN
+F 3 "~" H 5150 3950 50  0001 C CNN
+	1    5150 3950
+	1    0    0    -1
+$EndComp
+Wire Wire Line
+	5350 3950 5450 3950
+Wire Wire Line
+	5350 4050 5450 4050
+Text GLabel 5450 3950 2    50   Input ~ 0
 SDA
-Text GLabel 5500 4300 2    50   Input ~ 0
+Text GLabel 5450 4050 2    50   Input ~ 0
 SCL
 $Comp
@@
 Text Label 950  4350 0    50   ~ 0
 MSB
+$Comp
+L power:+5V #PWR0106
+U 1 1 5C5FBF14
+P 5550 2700
+F 0 "#PWR0106" H 5550 2550 50  0001 C CNN
+F 1 "+5V" H 5565 2873 50  0000 C CNN
+F 2 "" H 5550 2700 50  0001 C CNN
+F 3 "" H 5550 2700 50  0001 C CNN
+	1    5550 2700
+	1    0    0    -1
+$EndComp
+$Comp
+L power:GND #PWR0107
+U 1 1 5C5FBFB4
+P 5500 4350
+F 0 "#PWR0107" H 5500 4100 50  0001 C CNN
+F 1 "GND" H 5505 4177 50  0000 C CNN
+F 2 "" H 5500 4350 50  0001 C CNN
+F 3 "" H 5500 4350 50  0001 C CNN
+	1    5500 4350
+	1    0    0    -1
+$EndComp
+Wire Wire Line
+	5500 4350 5500 4150
+Wire Wire Line
+	5500 4150 5350 4150
+Wire Wire Line
+	5400 2800 5550 2800
+Wire Wire Line
+	5550 2800 5550 2700
+$Comp
+L power:+5V #PWR0108
+U 1 1 5C60D83D
+P 5500 3750
+F 0 "#PWR0108" H 5500 3600 50  0001 C CNN
+F 1 "+5V" H 5515 3923 50  0000 C CNN
+F 2 "" H 5500 3750 50  0001 C CNN
+F 3 "" H 5500 3750 50  0001 C CNN
+	1    5500 3750
+	1    0    0    -1
+$EndComp
+Wire Wire Line
+	5350 3850 5500 3850
+Wire Wire Line
+	5500 3850 5500 3750
+$Comp
+L power:GND #PWR0109
+U 1 1 5C611EC8
+P 5550 3200
+F 0 "#PWR0109" H 5550 2950 50  0001 C CNN
+F 1 "GND" H 5555 3027 50  0000 C CNN
+F 2 "" H 5550 3200 50  0001 C CNN
+F 3 "" H 5550 3200 50  0001 C CNN
+	1    5550 3200
+	1    0    0    -1
+$EndComp
+Wire Wire Line
+	5550 3200 5550 3000
+Wire Wire Line
+	5550 3000 5400 3000
 $EndSCHEMATC
